Commit message: Latest work

File: StickASM/urdf/StickASM.urdf (robot description, URDF)
Before this commit: robot StickASM, 17 links, 16 joints
Joints:
- joint BRFeet: origin xyz=0 -0.1 0.029473 rpy=3.1416 -1.5708 0 -> xyz=0 -0.1 0.029473 rpy=0 -1.5708 0
- joint FRFeet: origin xyz=0 -0.1 0.0248934676145698 rpy=3.14159263868863 -1.5707963267949 0 -> xyz=0 -0.1 0.0248934676145698 rpy=0 -1.5707963267949 0
